File: PCIexpress_x16_half/decap.kicad_sch (KiCad schematic)
At the start: 2 parts

Commit message: Added x2
added x2 cards
updated for KiCad 9
Parts:
- C1, C2: renamed from C?; value (none) -> 100n; footprint (none) -> Capacitor_SMD:C_0603_1608Metric
