File: PCIexpress_x16_half/term.kicad_sch (KiCad schematic)
At the start: 2 parts

Commit message: Added x2
added x2 cards
updated for KiCad 9
Parts:
- R1, R2: value (none) -> 49.9; footprint (none) -> Resistor_SMD:R_0603_1608Metric
